File: nist.sch (KiCad schematic (older format))
At the start: 35 parts

Commit message: added code
Parts:
- added U20, U24, U28, U32, U36, U40, U44, U48, U52, U56, U60, U64: 74LS273, symbol 74LS273
- gave numbers to parts that had none: 4
Connections:
- net labels added: CLK_U20, CLK_U24, CLK_U28, CLK_U32, CLK_U36, CLK_U40, CLK_U44, CLK_U48, CLK_U52, CLK_U56, CLK_U60, CLK_U64, ~MR
- wire segments 234 -> 360
Other:
- note removed: "to relay flipflops"
- moved on the sheet: R?, U11, U12, U14, U15, U?, U?A, U?B, U?C, U?D, U?E, U?F
